File: LightStripSensor/LightStripSensor.kicad_sch (KiCad schematic)
At the start: 14 parts, among them J1 LED_OUT 5.5x2.1, J2 DC_IN 12V 5.5x2.1, J3 HLK-LD2410B, Q1 IRLR7843, U1 ESP32-C3-SuperMini, U2 LM7805_TO220

Commit message: Update LightStripSensor
- Add footprint: Resistor, Capasitor, SMD _Esp32
- Design PCB LightStripSensor
Parts:
- C1, C4, C5: footprint (none) -> Capacitor_SMD:C_0805_2012Metric_Pad1.18x1.45mm_HandSolder
- C2, C3: footprint (none) -> Capacitor_SMD:C_Elec_8x10.2
- D1: value D_Schottky -> 3A; footprint (none) -> Diode_SMD:D_SMA_Handsoldering
- R1, R2: footprint (none) -> Resistor_SMD:R_0805_2012Metric_Pad1.20x1.40mm_HandSolder
Changed lines of the file:
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@@
 			)
 		)
-		(property "Footprint" ""
+		(property "Footprint" "Capacitor_SMD:C_Elec_8x10.2"
 			(at 82.55 110.49 0)
 			(hide yes)
@@
 			)
 		)
-		(property "Footprint" ""
+		(property "Footprint" "Resistor_SMD:R_0805_2012Metric_Pad1.20x1.40mm_HandSolder"
 			(at 58.42 154.94 0)
 			(hide yes)
@@
 			)
 		)
-		(property "Footprint" ""
+		(property "Footprint" "Capacitor_SMD:C_0805_2012Metric_Pad1.18x1.45mm_HandSolder"
 			(at 95.25 110.49 0)
 			(hide yes)
@@
 			)
 		)
-		(property "Footprint" ""
+		(property "Footprint" "Resistor_SMD:R_0805_2012Metric_Pad1.20x1.40mm_HandSolder"
 			(at 53.34 147.32 0)
 			(hide yes)
@@
 			)
 		)
-		(property "Footprint" ""
+		(property "Footprint" "Capacitor_SMD:C_0805_2012Metric_Pad1.18x1.45mm_HandSolder"
 			(at 41.91 110.49 0)
 			(hide yes)
@@
 			)
 		)
-		(property "Footprint" ""
+		(property "Footprint" "Capacitor_SMD:C_Elec_8x10.2"
 			(at 52.07 110.49 0)
 			(hide yes)
@@
 			)
 		)
-		(property "Footprint" ""
+		(property "Footprint" "Capacitor_SMD:C_0805_2012Metric_Pad1.18x1.45mm_HandSolder"
 			(at 102.87 147.32 0)
 			(hide yes)
@@
 			)
 		)
-		(property "Value" "D_Schottky"
+		(property "Value" "3A"
 			(at 96.52 148.336 90)
 			(show_name no)
@@
 			)
 		)
-		(property "Footprint" ""
+		(property "Footprint" "Diode_SMD:D_SMA_Handsoldering"
 			(at 99.06 147.32 0)
 			(hide yes)

Commit message: LightStripSensor: Add protection parts
Parts:
- removed U2: LM7805_TO220, Package_TO_SOT_SMD:TO-263-3_TabPin2, symbol Regulator_Linear:LM7805_TO220
- added D2: BZT52C15, Diode_SMD:D_SOD-123, symbol Device:D_Zener
- added D3: SMBJ15A, Diode_SMD:D_SMB, symbol Device:D_Zener
- added F1: 5A fast, Fuse:Fuse_2512_6332Metric_Pad1.52x3.35mm_HandSolder, symbol Device:Fuse
- added Q2: AOD4185, Package_TO_SOT_SMD:TO-252-2, symbol Transistor_FET:Q_PMOS_GDS
- added R3: 10k, Resistor_SMD:R_0805_2012Metric_Pad1.20x1.40mm_HandSolder, symbol Device:R_Small_US
- added U2: L7805 (TO-263), Package_TO_SOT_SMD:TO-263-3_TabPin2, symbol Regulator_Linear:L7805
Connections:
- net GND: now also D3.2 (A), R3.2, U2.2 (GND)
- net VDD: now also U2.3 (OUT)
- net V_in: now also D2.1 (K), D3.1 (K), Q2.3 (S), U2.1 (IN); no longer J2.1
- new net: F1.1, J2.1
- new net: D2.2 (A), Q2.1 (G), R3.1
- new net: F1.2, Q2.2 (D)
Other:
- moved on the sheet: J1

Commit message: Update SCH/PCB
- Delete Mosfet and Zenner
- Design PCB
Parts:
- removed D2: BZT52C15, Diode_SMD:D_SOD-123, symbol Device:D_Zener
- removed Q2: AOD4185, Package_TO_SOT_SMD:TO-252-2, symbol Transistor_FET:Q_PMOS_GDS
- removed R3: 10k, Resistor_SMD:R_0805_2012Metric_Pad1.20x1.40mm_HandSolder, symbol Device:R_Small_US
- F1: value 5A fast -> 7A fast; footprint Fuse:Fuse_2512_6332Metric_Pad1.52x3.35mm_HandSolder -> Fuse:Fuse_1812_4532Metric_Pad1.30x3.40mm_HandSolder
Connections:
- net V_in: now also F1.2
Other:
- moved on the sheet: D3

Commit message: Update Sch and PCB
- sch add capacitor  100nf
-  pcb redesign: Reroute
Parts:
- added C6: 100n, Capacitor_SMD:C_0805_2012Metric_Pad1.18x1.45mm_HandSolder, symbol Device:C_Small
Connections:
- net GND: now also C6.2
- net VDD: now also C6.1
Changed lines of the file:
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@@
+	)
+	(junction
+		(at 95.25 115.57)
+		(diameter 0)
+		(color 0 0 0 0)
 	)
 	(junction
@@
 	(wire
 		(pts
+			(xy 95.25 115.57) (xy 109.22 115.57)
+		)
+		(stroke
+			(width 0)
+			(type default)
+		)
+	)
+	(wire
+		(pts
 			(xy 102.87 143.51) (xy 99.06 143.51)
 		)
@@
 	(wire
 		(pts
+			(xy 95.25 107.95) (xy 109.22 107.95)
+		)
+		(stroke
+			(width 0)
+			(type default)
+		)
+	)
+	(wire
+		(pts
 			(xy 76.2 107.95) (xy 82.55 107.95)
 		)
@@
 		(pts
 			(xy 82.55 115.57) (xy 68.58 115.57)
+		)
+		(stroke
+			(width 0)
+			(type default)
+		)
+	)
+	(wire
+		(pts
+			(xy 109.22 113.03) (xy 109.22 115.57)
 		)
 		(stroke
@@
 					(unit 1)
 				)
+			)
+		)
+	)
+	(symbol
+		(lib_id "Device:C_Small")
+		(at 109.22 110.49 0)
+		(unit 1)
+		(body_style 1)
+		(exclude_from_sim no)
+		(in_bom yes)
+		(on_board yes)
+		(in_pos_files yes)
+		(dnp no)
+		(fields_autoplaced yes)
+		(property "Reference" "C6"
+			(at 111.76 109.2262 0)
+			(show_name no)
+			(do_not_autoplace no)
+			(effects
+				(font
+					(size 1.27 1.27)
+				)
+				(justify left)
+			)
+		)
+		(property "Value" "100n"
+			(at 111.76 111.7662 0)
+			(show_name no)
+			(do_not_autoplace no)
+			(effects
+				(font
+					(size 1.27 1.27)
+				)
+				(justify left)
+			)
+		)
+		(property "Footprint" "Capacitor_SMD:C_0805_2012Metric_Pad1.18x1.45mm_HandSolder"
+			(at 109.22 110.49 0)
+			(hide yes)
+			(show_name no)
+			(do_not_autoplace no)
+			(effects
+				(font
+					(size 1.27 1.27)
+				)
+			)
+		)
+		(property "Datasheet" ""
+			(at 109.22 110.49 0)
+			(hide yes)
+			(show_name no)
+			(do_not_autoplace no)
+			(effects
+				(font
+					(size 1.27 1.27)
+				)
+			)
+		)
+		(property "Description" "Unpolarized capacitor, small symbol"
+			(at 109.22 110.49 0)
+			(hide yes)
+			(show_name no)
+			(do_not_autoplace no)
+			(effects
+				(font
+					(size 1.27 1.27)
+				)
+			)
+		)
+		(pin "1"
+		)
+		(pin "2"
+		)
+		(instances
+			(project "LightStripSensor"
+				(path "/4228bc61-6b6e-4a67-a78d-24cb95585443"
+					(reference "C6")
+					(unit 1)
+				)
